File: ElectronicPsychicSchematics/ThePsychic.sch (KiCad schematic (older format))
At the start: 25 parts, among them SW1 1, SW10 6, SW11 9, SW12 #, SW13 A, SW14 B, SW15 C, SW16 D, SW2 4, SW3 7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

Commit message: Remove incriminating comments and save as Assistant.ino to share without revealing too much secret
Parts:
- U0: value Any two-digit 6-segment -> Any two-digit Common Anode
Changed lines of the file:
@@
 P 9900 4700
 F 0 "U0" H 9900 5367 50  0001 C CNN
-F 1 "Any two-digit 6-segment" H 9900 5275 50  0000 C CNN
+F 1 "Any two-digit Common Anode" H 9900 5275 50  0000 C CNN
 F 2 "Display:HDSM-441B_HDSM-443B" H 9900 4100 50  0001 C CNN
 F 3 "https://docs.broadcom.com/docs/AV02-1589EN" H 9680 4800 50  0001 C CNN

Commit message: Fixed schematic error
Parts:
- removed U0: Any two-digit Common Anode, Display:HDSM-441B_HDSM-443B, symbol Display_Character:HDSM-441B
- added U?: Any_2Digit_7Segment, Display:HDSM-441B_HDSM-443B, symbol ElectronicPsychicSchematics-cache:Any_2Digit_7Segment
Connections:
- wire segments 98 -> 96
Other:
- moved on the sheet: All1
Changed lines of the file:
@@
 $EndDescr
-$Comp
-L Display_Character:HDSM-441B U0
-U 1 1 5FB1882B
-P 9900 4700
-F 0 "U0" H 9900 5367 50  0001 C CNN
-F 1 "Any two-digit Common Anode" H 9900 5275 50  0000 C CNN
-F 2 "Display:HDSM-441B_HDSM-443B" H 9900 4100 50  0001 C CNN
-F 3 "https://docs.broadcom.com/docs/AV02-1589EN" H 9680 4800 50  0001 C CNN
-	1    9900 4700
-	1    0    0    -1
-$EndComp
 $Comp
 L MCU_Module:Arduino_Nano_v3.x A1
@@
 L Device:R_Small_US R2
 U 1 1 5FB22D5D
+P 9100 5200
+F 0 "R2" V 8987 5200 50  0001 C CNN
+F 1 "R_Small_US" V 8986 5200 50  0001 C CNN
+F 2 "" H 9100 5200 50  0001 C CNN
+F 3 "~" H 9100 5200 50  0001 C CNN
+	1    9100 5200
+	0    1    1    0
+$EndComp
+$Comp
+L Device:R_Small_US All1
+U 1 1 5FB26493
 P 9100 4600
-F 0 "R2" V 8987 4600 50  0001 C CNN
-F 1 "R_Small_US" V 8986 4600 50  0001 C CNN
+F 0 "All1" V 8900 4600 50  0000 C CNN
+F 1 "220" V 8987 4600 50  0000 C CNN
 F 2 "" H 9100 4600 50  0001 C CNN
 F 3 "~" H 9100 4600 50  0001 C CNN
 	1    9100 4600
-	0    1    1    0
-$EndComp
-$Comp
-L Device:R_Small_US All1
-U 1 1 5FB26493
-P 9100 4400
-F 0 "All1" V 8900 4400 50  0000 C CNN
-F 1 "220" V 8987 4400 50  0000 C CNN
-F 2 "" H 9100 4400 50  0001 C CNN
-F 3 "~" H 9100 4400 50  0001 C CNN
-	1    9100 4400
 	0    1    1    0
 $EndComp
@@
 $EndComp
 Wire Wire Line
-	9300 4400 9200 4400
-Wire Wire Line
 	9300 4800 9200 4800
 Wire Wire Line
@@
 	8450 5000 9000 5000
 Wire Wire Line
-	9000 4400 8900 4400
-Wire Wire Line
-	8900 4400 8900 5200
-Wire Wire Line
-	8900 5200 8450 5200
-Wire Wire Line
 	8450 5100 9000 5100
 Wire Wire Line
-	10500 5000 10700 5000
-Wire Wire Line
-	10700 5000 10700 5600
+	10500 5200 10700 5200
+Wire Wire Line
+	10700 5200 10700 5600
 Wire Wire Line
 	10700 5600 8450 5600
 Wire Wire Line
-	10500 5100 10600 5100
-Wire Wire Line
-	10600 5100 10600 5700
+	10500 5300 10600 5300
+Wire Wire Line
+	10600 5300 10600 5700
 Wire Wire Line
 	10600 5700 8450 5700
-$Comp
-L power:GND #PWR0102
-U 1 1 5FB2F302
-P 8900 6050
-F 0 "#PWR0102" H 8900 5800 50  0001 C CNN
-F 1 "GND" H 8905 5877 50  0000 C CNN
-F 2 "" H 8900 6050 50  0001 C CNN
-F 3 "" H 8900 6050 50  0001 C CNN
-	1    8900 6050
-	1    0    0    -1
-$EndComp
 Wire Wire Line
 	8500 5500 8450 5500
-NoConn ~ 9300 4500
+NoConn ~ 9300 5300
 NoConn ~ 8450 4400
 NoConn ~ 8450 4500
@@
 L power:PWR_FLAG #FLG01
 U 1 1 5FB43413
-P 9150 6050
-F 0 "#FLG01" H 9150 6125 50  0001 C CNN
-F 1 "PWR_FLAG" H 9150 6223 50  0000 C CNN
-F 2 "" H 9150 6050 50  0001 C CNN
-F 3 "~" H 9150 6050 50  0001 C CNN
-	1    9150 6050
+P 8600 6050
+F 0 "#FLG01" H 8600 6125 50  0001 C CNN
+F 1 "PWR_FLAG" H 8600 6223 50  0000 C CNN
+F 2 "" H 8600 6050 50  0001 C CNN
+F 3 "~" H 8600 6050 50  0001 C CNN
+	1    8600 6050
 	1    0    0    -1
 $EndComp
@@
 L power:GND #PWR01
 U 1 1 5FB44C53
-P 9150 6050
-F 0 "#PWR01" H 9150 5800 50  0001 C CNN
-F 1 "GND" H 9155 5877 50  0000 C CNN
-F 2 "" H 9150 6050 50  0001 C CNN
-F 3 "" H 9150 6050 50  0001 C CNN
-	1    9150 6050
+P 8600 6050
+F 0 "#PWR01" H 8600 5800 50  0001 C CNN
+F 1 "GND" H 8605 5877 50  0000 C CNN
+F 2 "" H 8600 6050 50  0001 C CNN
+F 3 "" H 8600 6050 50  0001 C CNN
+	1    8600 6050
 	1    0    0    -1
 $EndComp
@@
 	6350 4850 6350 5250
 NoConn ~ 8500 5500
+$Comp
+L ElectronicPsychicSchematics-cache:Any_2Digit_7Segment U?
+U 1 1 5FB563C1
+P 9900 4900
+F 0 "U?" H 9900 5567 50  0000 C CNN
+F 1 "Any_2Digit_7Segment" H 9900 5476 50  0000 C CNN
+F 2 "Display:HDSM-441B_HDSM-443B" H 9900 4300 50  0001 C CNN
+F 3 "" H 9680 5000 50  0001 C CNN
+	1    9900 4900
+	1    0    0    -1
+$EndComp
+Wire Wire Line
+	8450 5200 9000 5200
+Wire Wire Line
+	9200 5200 9300 5200
 $EndSCHEMATC

Commit message: Source cleanup
Parts:
- U1: renamed from U?; value Any_2Digit_7Segment -> Common Anode 7-Segment; symbol ElectronicPsychicSchematics-cache:Any_2Digit_7Segment -> ThePsychic-rescue:Any_2Digit_7Segment-ElectronicPsychicSchematics-cache
Connections:
- net at A1.15 (D12): now also U1.5 (CA_DIG0); no longer U1.10 (CA_DIG1)
- net at A1.16 (D13): now also U1.10 (CA_DIG1); no longer U1.5 (CA_DIG2)
Changed lines of the file:
@@
 	8450 5100 9000 5100
 Wire Wire Line
-	10500 5200 10700 5200
-Wire Wire Line
-	10700 5200 10700 5600
-Wire Wire Line
-	10700 5600 8450 5600
-Wire Wire Line
-	10500 5300 10600 5300
-Wire Wire Line
-	10600 5300 10600 5700
-Wire Wire Line
-	10600 5700 8450 5700
+	10100 5500 10100 5600
+Wire Wire Line
+	10100 5600 8450 5600
+Wire Wire Line
+	9750 5500 9750 5700
+Wire Wire Line
+	9750 5700 8450 5700
 Wire Wire Line
 	8500 5500 8450 5500
@@
 NoConn ~ 8500 5500
 $Comp
-L ElectronicPsychicSchematics-cache:Any_2Digit_7Segment U?
+L ThePsychic-rescue:Any_2Digit_7Segment-ElectronicPsychicSchematics-cache U1
 U 1 1 5FB563C1
 P 9900 4900
-F 0 "U?" H 9900 5567 50  0000 C CNN
-F 1 "Any_2Digit_7Segment" H 9900 5476 50  0000 C CNN
+F 0 "U1" H 9900 5567 50  0001 C CNN
+F 1 "Common Anode 7-Segment" H 9900 5476 50  0000 C CNN
 F 2 "Display:HDSM-441B_HDSM-443B" H 9900 4300 50  0001 C CNN
 F 3 "" H 9680 5000 50  0001 C CNN
